Commit message: add lidar and imu sensors

File: urdf/diff_robot.urdf (robot description, URDF)
Before this commit: robot diff_robot, 7 links, 6 joints
Links:
- link imu_link: geometry visual box size=0.01 0.01 0.01
- link lidar_link: geometry collision cylinder length=0.05 radius=0.05; visual cylinder length=0.05 radius=0.1
Joints:
- joint base_joint: origin xyz=0.0 0.0 0.1 rpy=0.0 0.0 0.0 -> xyz=0.0 0.0 0.05 rpy=0.0 0.0 0.0
